File: dspic.kicad_sch (KiCad schematic)
At the start: 18 parts, among them U4 DSPIC33FJ128GP204

Commit message: update layers
Parts:
- added D8, D9: LED, LED_SMD:LED_0603_1608Metric, symbol Device:LED
- added R17, R18: 50, Resistor_SMD:R_0603_1608Metric, symbol Device:R
Connections:
- net GND: now also D8.1 (K), D9.1 (K)
- net B10: now reaches U4.8 (PGED2/EMCD2/RP10/CN16/PMD2/RB10)
- net B10: now also R17.2
- net B11: now reaches U4.9 (PGEC2/RP11/CN15/PMD1/RB11)
- net B11: now also R18.2
- new net: D9.2 (A), R18.1
- new net: D8.2 (A), R17.1
Other:
- moved on the sheet: D2, D3, D4, D5, D6, D7, R11, R12, R13, R14, R15, R16

Commit message: curtis changes
Parts:
- D2, D3, D4, D5, D6, D7, D8, D9: footprint LED_SMD:LED_0603_1608Metric -> LED_SMD:LED_0805_2012Metric
- R11, R12, R13, R14, R15, R16, R17, R18: value 50 -> 1k
Changed lines of the file:
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@@
 			)
 		)
-		(property "Footprint" "LED_SMD:LED_0603_1608Metric"
+		(property "Footprint" "LED_SMD:LED_0805_2012Metric"
 			(at 245.11 99.06 0)
 			(effects
@@
 			)
 		)
-		(property "Value" "50"
+		(property "Value" "1k"
 			(at 237.744 84.836 0)
 			(effects
@@
 			)
 		)
-		(property "Value" "50"
+		(property "Value" "1k"
 			(at 203.454 84.836 0)
 			(effects
@@
 			)
 		)
-		(property "Footprint" "LED_SMD:LED_0603_1608Metric"
+		(property "Footprint" "LED_SMD:LED_0805_2012Metric"
 			(at 222.25 99.06 0)
 			(effects
@@
 			)
 		)
-		(property "Footprint" "LED_SMD:LED_0603_1608Metric"
+		(property "Footprint" "LED_SMD:LED_0805_2012Metric"
 			(at 199.39 99.06 0)
 			(effects
@@
 			)
 		)
-		(property "Footprint" "LED_SMD:LED_0603_1608Metric"
+		(property "Footprint" "LED_SMD:LED_0805_2012Metric"
 			(at 210.82 99.06 0)
 			(effects
@@
 			)
 		)
-		(property "Footprint" "LED_SMD:LED_0603_1608Metric"
+		(property "Footprint" "LED_SMD:LED_0805_2012Metric"
 			(at 176.53 99.06 0)
 			(effects
@@
 			)
 		)
-		(property "Value" "50"
+		(property "Value" "1k"
 			(at 180.594 84.836 0)
 			(effects
@@
 			)
 		)
-		(property "Footprint" "LED_SMD:LED_0603_1608Metric"
+		(property "Footprint" "LED_SMD:LED_0805_2012Metric"
 			(at 165.1 99.06 0)
 			(effects
@@
 			)
 		)
-		(property "Footprint" "LED_SMD:LED_0603_1608Metric"
+		(property "Footprint" "LED_SMD:LED_0805_2012Metric"
 			(at 233.68 99.06 0)
 			(effects
@@
 			)
 		)
-		(property "Footprint" "LED_SMD:LED_0603_1608Metric"
+		(property "Footprint" "LED_SMD:LED_0805_2012Metric"
 			(at 187.96 99.06 0)
 			(effects
@@
 			)
 		)
-		(property "Value" "50"
+		(property "Value" "1k"
 			(at 249.174 84.836 0)
 			(effects
@@
 			)
 		)
-		(property "Value" "50"
+		(property "Value" "1k"
 			(at 192.024 84.836 0)
 			(effects
@@
 			)
 		)
-		(property "Value" "50"
+		(property "Value" "1k"
 			(at 169.164 84.836 0)
 			(effects
@@
 			)
 		)
-		(property "Value" "50"
+		(property "Value" "1k"
 			(at 226.314 84.836 0)
 			(effects
@@
 			)
 		)
-		(property "Value" "50"
+		(property "Value" "1k"
 			(at 214.884 84.836 0)
 			(effects

Commit message: removed pad via
Connections:
- net GND: now also U4.16 (AVSS)
Changed lines of the file:
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@@
+	)
+	(junction
+		(at 86.36 142.24)
+		(diameter 0)
+		(color 0 0 0 0)
 	)
 	(junction
@@
 		)
 		(stroke
+			(width 0)
+			(type default)
+		)
+	)
+	(wire
+		(pts
+			(xy 86.36 142.24) (xy 91.44 142.24)
+		)
+		(stroke
